File: HW2/433_PCB/ME433_board.sch (EAGLE design)
At the start: 14 parts, among them J1 USB_MINI-B_SMT, Y1 NU32V7_RESONATORSMD

Commit message: board design and gerber generation
Parts:
- added J3, J4: (no value), SparkFun-Connectors:CONN_08"
- added LED2: Green, ME433_library:LEDSML0603
- added R2: 330Ω, ME433_library:R-US_R0603
- added R3, R4: 10kΩ, ME433_library:R-US_R0603
- added RESET: RESET, ME433_library:NU32V7_MOM_SW
- added USER: USER, ME433_library:NU32V7_MOM_SW
- C5: value (none) -> 0.1uF
- LED1: device ME433_library:LEDP-LCC-2-BACK -> ME433_library:LEDSML0603
- renumbered J1 to MINIUSB, U$2 to PWR_SW, Y1 to RESONATOR
Connections:
- new net N$2: LED2.C, R2.2
- net +3V3: now also J4.2, R3.2, R4.2
- net +5V: now also J3.2
- net A0: now also J4.8
- net A1: now also J4.7
- net A4/LED: now also J4.3, LED2.A
- net B13: now also J3.6
- net B14: now also J3.7
- net B15: now also J3.8
- net B2: now also J4.6
- net B3: now also J4.5
- net B4/USER: now also J4.4, R3.1, USER.1.B
- net B7: now also J3.3
- net B8: now also J3.4
- net B9: now also J3.5
- net GND: now also J3.1, J4.1, R2.1, RESET.2.A, USER.2.A
- net MCLR: now also R4.1, RESET.1.B
